File: stm32breakout.kicad_sch (KiCad schematic)
At the start: 42 parts, among them J1 USB_C_Receptacle_USB2.0_16P, J2 GPIO_LEFT, J3 GPIO_RIGHT, J4 SWD, SW1 NRST, SW2 BOOT0, U1 STM32F103C8Tx, U2 AP2112K-3.3, Y1 8MHz, Y2 32.768kHz

Commit message: Finish 2-layer routing and export JLCPCB fab files.
DRC is 0 geometry / 0 unconnected and ERC is 0. Analog filter
(FB1/C8/C9) is left of the MCU so last-mile +3V3/+3V3A and
NRST-to-J4 clear. Gerbers, LCSC BOM, and pick-and-place are in fab/.
Parts:
- C1, C4: LCSC (none) -> C19702
- C10, C15, C5, C6, C7, C8: LCSC (none) -> C14663
- C11, C12: LCSC (none) -> C1645
- C13, C14: LCSC (none) -> C1647
- C2, C3, C9: LCSC (none) -> C15849
- D1: LCSC (none) -> C72043
- D2: LCSC (none) -> C72041
- FB1: LCSC (none) -> C23611
- J1: LCSC (none) -> C165948
- J2, J3: LCSC (none) -> C124378
- J4: LCSC (none) -> C124376
- R1, R2: LCSC (none) -> C23181
- R10: LCSC (none) -> C25803
- R3, R4: LCSC (none) -> C17561
- R5, R6, R7: LCSC (none) -> C25804
- R8, R9: LCSC (none) -> C21190
- SW1, SW2: LCSC (none) -> C318884
- U1: LCSC (none) -> C8734
- U2: LCSC (none) -> C51118
- Y1: LCSC (none) -> C9002
- Y2: LCSC (none) -> C32346
